Commit message: feat(control-studio): industrial CAD visual overhaul, 6-DOF Euler orientation, wrist presets, and comprehensive Polish localization
- Upgrade Control Studio with soft neutral precision CAD styling, bevel tokens, and 100vh zero-scroll layout
- Add vernier scale dual-markers (live vs ghost) and animated SVG gripper jaw indicator
- Enhance Three.js viewport with calibrated studio lighting, PBR materials, polar CAD grid, and 2D-3D joint hover highlighting
- Implement 6-DOF Euler orientation with orbital yaw tracking, 7 wrist presets (W0-W6), and J5 limit alignment (-120°..+120°)
- Overhaul bilingual English/Polish localization across UI and documentation with natural industrial robotics terminology
- Expand automated test suite to 618/618 passing tests across 25 suites
- Add PCB layout concept, wiring diagrams, and perfboard cutting plans

File: WebControl/urdf/stppe_zlozenie_nowe.urdf (robot description, URDF)
Before this commit: robot stppe_zlozenie_nowe, 7 links, 6 joints
Joints:
- joint joint_5: limit lower=-1.570796 upper=1.570796 effort=100 velocity=100 -> lower=-2.094395 upper=2.094395 effort=100 velocity=100
